File: kicad/power-distribution/power-distribution.kicad_sch (KiCad schematic)
At the start: 0 parts

Commit message: started with pd schem
Other:
- company: (none) -> Rover to Mars (R2M)
- title: (none) -> Power Distribution
Changed lines of the file:
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@@
 	(paper "A4")
 	(title_block
+		(title "Power Distribution")
 		(date "2024-05-12")
+		(rev "A")
+		(company "Rover to Mars (R2M)")
+		(comment 1 "Leandro Ebner")
+		(comment 3 "Ravensburg-Weingarten University")
 	)
 	(sheet
-		(at 36.83 99.06)
+		(at 83.82 52.07)
 		(size 12.7 3.81)
 		(fields_autoplaced yes)
@@
 		)
 		(property "Sheetname" "primary-pd"
-			(at 36.83 98.3484 0)
+			(at 83.82 51.3584 0)
 			(effects
 				(font
@@
 		)
 		(property "Sheetfile" "primary-pd.kicad_sch"
-			(at 36.83 103.4546 0)
+			(at 83.82 56.4646 0)
 			(effects
 				(font
@@
 	)
 	(sheet
-		(at 68.58 99.06)
+		(at 104.14 50.8)
 		(size 12.7 3.81)
 		(fields_autoplaced yes)
@@
 		)
 		(property "Sheetname" "secondary-pd"
-			(at 68.58 98.3484 0)
+			(at 104.14 50.0884 0)
 			(effects
 				(font
@@
 		)
 		(property "Sheetfile" "secondary-pd.kicad_sch"
-			(at 68.58 103.4546 0)
+			(at 104.14 55.1946 0)
 			(effects
 				(font
