File: kicad/power-distribution/secondary-pd.kicad_sch (KiCad schematic)
At the start: 0 parts

Commit message: started with pd schem
Other:
- company: (none) -> Rover to Mars (R2M)
- title: (none) -> Power Distribution
Changed lines of the file:
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@@
 	(paper "A4")
 	(title_block
+		(title "Power Distribution")
 		(date "2024-05-12")
+		(rev "A")
+		(company "Rover to Mars (R2M)")
+		(comment 1 "Leandro Ebner")
+		(comment 3 "Ravensburg-Weingarten University")
 	)
 )
